File: pcb/acq_apd.sch (KiCad schematic (older format))
At the start: 15 parts, among them P12 EPV, U9 LT3571

Commit message: pcb: Update to the current iteration
Looks like I forgot to commit the changes made for manufacturing...
Parts:
- C36: value 100n -> 100n/200V; footprint Resistors_SMD:R_0402 -> Resistors_SMD:R_0805
- JP3: value Jumper_NO_Small -> DNP
- U9: value LT3571 -> LT3571EUD
Changed lines of the file:
@@
 EESchema Schematic File Version 2
+LIBS:pcb-rescue
 LIBS:power
 LIBS:device
@@
 P 5700 4125
 F 0 "U9" H 5400 3575 59  0000 C CNN
-F 1 "LT3571" H 5500 3725 59  0000 C CNN
+F 1 "LT3571EUD" H 5700 3775 59  0000 C CNN
 F 2 "Housings_DFN_QFN:QFN-16-1EP_3x3mm_Pitch0.5mm" H 5700 4125 197 0001 C CNN
 F 3 "" H 5700 4125 197 0000 C CNN
@@
 P 6825 3900
 F 0 "C36" H 6835 3970 50  0000 L CNN
-F 1 "100n" H 6835 3820 50  0000 L CNN
-F 2 "Resistors_SMD:R_0402" H 6825 3900 50  0001 C CNN
+F 1 "100n/200V" H 6835 3820 50  0000 L CNN
+F 2 "Resistors_SMD:R_0805" H 6825 3900 50  0001 C CNN
 F 3 "" H 6825 3900 50  0000 C CNN
 	1    6825 3900
@@
 P 7025 3625
 F 0 "JP3" H 7025 3705 50  0000 C CNN
-F 1 "Jumper_NO_Small" H 7035 3565 50  0001 C CNN
+F 1 "DNP" H 7035 3565 50  0001 C CNN
 F 2 "Resistors_SMD:R_0402" H 7025 3625 50  0001 C CNN
 F 3 "" H 7025 3625 50  0000 C CNN
