File: pcb/acq_mcu.sch (KiCad schematic (older format))
At the start: 30 parts, among them P11 EPV, P3 SWD, P4 SWC, P5 USB_OTG, U6 STM32F302KxU, U7 NCP700B, U8 501HCA12M0000DAG

Commit message: pcb: Update to the current iteration
Looks like I forgot to commit the changes made for manufacturing...
Parts:
- D1, D2: symbol LED -> LED-RESCUE-pcb
- P5: footprint Connect:USB_Micro-B -> footprints:USB_Micro-B; symbol USB_OTG -> USB_OTG-RESCUE-pcb
- U6: value STM32F302KxU -> STM32F302K8U6
- U7: value NCP700B -> NCP700BSN33T1G
- U8: value 501HCA12M0000DAG -> QX333A12.00000B15M; footprint footprints:501HCA_2.5x2 -> footprints:QX333A
Changed lines of the file:
@@
 EESchema Schematic File Version 2
+LIBS:pcb-rescue
 LIBS:power
 LIBS:device
@@
 U 1 1 572D793B
 P 10025 5425
-F 0 "U7" H 10125 4975 60  0000 C CNN
-F 1 "NCP700B" H 10275 5075 60  0000 C CNN
+F 0 "U7" H 10150 5100 60  0000 C CNN
+F 1 "NCP700BSN33T1G" H 10000 5725 60  0000 C CNN
 F 2 "TO_SOT_Packages_SMD:SOT-23-5" H 10975 4675 60  0001 C CNN
 F 3 "" H 10975 4675 60  0000 C CNN
@@
 Connection ~ 10900 5275
 $Comp
-L USB_OTG P5
+L USB_OTG-RESCUE-pcb P5
 U 1 1 572D7984
 P 8725 3675
 F 0 "P5" H 9050 3550 50  0000 C CNN
 F 1 "USB_OTG" H 8725 3875 50  0000 C CNN
-F 2 "Connect:USB_Micro-B" V 8675 3575 50  0001 C CNN
+F 2 "footprints:USB_Micro-B" V 8675 3575 50  0001 C CNN
 F 3 "" V 8675 3575 50  0000 C CNN
 	1    8725 3675
@@
 P 3550 5150
 F 0 "U6" H 1250 4100 60  0000 C CNN
-F 1 "STM32F302KxU" H 2750 4100 60  0000 C CNN
+F 1 "STM32F302K8U6" H 2750 4100 60  0000 C CNN
 F 2 "Housings_DFN_QFN:QFN-32-1EP_5x5mm_Pitch0.5mm" H 3500 4750 60  0001 C CNN
 F 3 "" H 3500 4750 60  0000 C CNN
@@
 P 10150 4175
 F 0 "U8" H 10450 3925 60  0000 C CNN
-F 1 "501HCA12M0000DAG" V 9775 4175 39  0000 C CNN
-F 2 "footprints:501HCA_2.5x2" H 9600 3675 60  0001 C CNN
+F 1 "QX333A12.00000B15M" V 9775 4175 39  0000 C CNN
+F 2 "footprints:QX333A" H 9600 3675 60  0001 C CNN
 F 3 "" H 9600 3675 60  0000 C CNN
 	1    10150 4175
@@
 $EndComp
 $Comp
-L LED D1
+L LED-RESCUE-pcb D1
 U 1 1 572E565A
 P 9475 2450
+AR Path="/572E565A" Ref="D1"  Part="1"
+AR Path="/572D32D1/572E565A" Ref="D1"  Part="1"
 F 0 "D1" H 9475 2550 50  0000 C CNN
 F 1 "LED" H 9475 2350 50  0000 C CNN
@@
 LED
 $Comp
-L LED D2
+L LED-RESCUE-pcb D2
 U 1 1 5731EF1F
 P 9800 2450
+AR Path="/5731EF1F" Ref="D2"  Part="1"
+AR Path="/572D32D1/5731EF1F" Ref="D2"  Part="1"
 F 0 "D2" H 9800 2550 50  0000 C CNN
 F 1 "LED" H 9800 2350 50  0000 C CNN
